Commit message: cambios menores en posicion de ruedas

File: install/practica1/share/practica1/urdf/robotito.urdf (robot description, URDF)
Before this commit: robot robotito, 4 links, 3 joints
Joints:
- joint caster_joint: origin xyz=0.15 0 -0.05 -> xyz=0.15 0 -0.11
- joint left_wheel_joint: origin xyz=-0.1 0.17 0 -> xyz=-0.1 0.18 0
- joint right_wheel_joint: origin xyz=-0.1 -0.17 0 -> xyz=-0.1 -0.18 0

File: src/practica1/urdf/robotito.urdf (robot description, URDF)
Before this commit: robot robotito, 4 links, 3 joints
Joints:
- joint caster_joint: origin xyz=0.15 0 -0.05 -> xyz=0.15 0 -0.105
- joint left_wheel_joint: origin xyz=-0.1 0.17 0 -> xyz=-0.1 0.1705 0
- joint right_wheel_joint: origin xyz=-0.1 -0.17 0 -> xyz=-0.1 -0.1705 0

Commit message: cambios de las ruedas

File: install/practica1/share/practica1/urdf/robotito.urdf (robot description, URDF)
Before this commit: robot robotito, 4 links, 3 joints
Links:
- link caster_wheel: geometry collision sphere radius=0.025; visual sphere radius=0.025
- link left_wheel: geometry collision cylinder length=0.04 radius=0.1; visual cylinder length=0.04 radius=0.1
- link right_wheel: geometry collision cylinder length=0.04 radius=0.1; visual cylinder length=0.04 radius=0.1
Joints:
- joint caster_joint: origin xyz=0.15 0 -0.11 -> xyz=0.15 0 -0.075
- joint left_wheel_joint: origin xyz=-0.1 0.18 0 -> xyz=-0.1 0.1705 0
- joint right_wheel_joint: origin xyz=-0.1 -0.18 0 -> xyz=-0.1 -0.1705 0

File: src/practica1/urdf/robotito.urdf (robot description, URDF)
Before this commit: robot robotito, 4 links, 3 joints
Links:
- link caster_wheel: geometry collision sphere radius=0.025; visual sphere radius=0.025
- link left_wheel: geometry collision cylinder length=0.04 radius=0.1; visual cylinder length=0.04 radius=0.1
- link right_wheel: geometry collision cylinder length=0.04 radius=0.1; visual cylinder length=0.04 radius=0.1
Joints:
- joint caster_joint: origin xyz=0.15 0 -0.105 -> xyz=0.15 0 -0.075
