Commit message: camera rgb added

File: install/practica1/share/practica1/urdf/camera.xacro (robot description, xacro)
@@ -1,73 +1 @@
-<?xml version="1.0"?>
-<robot xmlns:xacro="http://www.ros.org/wiki/xacro" >
-    <joint name="camera_mast_joint" type="fixed">
-        <parent link="base_link"/>
-        <child link="camera_mast"/>
-        <origin xyz="0.10 0 0.20" rpy="0 0 0"/>
-    </joint>
-    <link name="camera_mast">
-        <visual>
-            <geometry>
-                <cylinder radius="0.02" length="0.30"/>
-            </geometry>
-            <material name="white"/>
-        </visual>
-        <collision>
-            <geometry>
-                <cylinder radius="0.02" length="0.30"/>
-            </geometry>
-        </collision>
-        <xacro:inertial_cylinder mass="0.05" length="0.30" radius="0.02">
-            <origin xyz="0 0 0" rpy="0 0 0"/>
-        </xacro:inertial_cylinder>
-    </link>
-    <joint name="camera_joint" type="fixed">
-        <parent link="camera_mast"/>
-        <child link="camera_link"/>
-        <origin xyz="0.02 0 0.15" rpy="0 0 0"/>
-    </joint>
-    <link name="camera_link">
-        <visual>
-            <geometry>
-                <box size="0.05 0.05 0.05"/>
-            </geometry>
-            <material name="blue"/>
-        </visual>
-        <collision>
-            <geometry>
-                <box size="0.05 0.05 0.05"/>
-            </geometry>
-        </collision>
-        <xacro:inertial_box mass="0.05" x="0.05" y="0.05" z="0.05">
-            <origin xyz="0 0 0" rpy="0 0 0"/>
-        </xacro:inertial_box>
-    </link>
-    <joint name="camera_optical_joint" type="fixed">
-        <origin xyz="0 0 0" rpy="-1.5708 0 -1.5708"/>
-        <parent link="camera_link"/>
-        <child link="camera_link_optical"/>
-    </joint>
-    <link name="camera_link_optical"></link>
-    <gazebo reference="camera_link">
-        <material>Gazebo/Blue</material>
-        <sensor name="camera" type="camera">
-            <pose> 0 0 0 0 0 0 </pose>
-            <visualize>true</visualize>
-            <update_rate>30.0</update_rate>
-            <camera>
-                <horizontal_fov>1.3962634</horizontal_fov>
-                <image>
-                    <width>800</width>
-                    <height>800</height>
-                    <format>R8G8B8</format>
-                </image>
-                <clip>
-                    <near>0.02</near>
-                    <far>300</far>
-                </clip>
-            </camera>
-            <topic>camera/image_raw</topic>
-            <gz_frame_id>camera_link_optical</gz_frame_id>
-        </sensor>
-    </gazebo>
-</robot>
+/ros2_ws_multirobots/src/practica1/urdf/camera.xacro

File: install/practica1/share/practica1/urdf/gazebo_control.xacro (robot description, xacro)
@@ -1,32 +1 @@
-<?xml version="1.0"?>
-<robot xmlns:xacro="http://www.ros.org/wiki/xacro">
-    <gazebo reference="caster_wheel">
-        <mu1 value="0.1" />
-        <mu2 value="0.1" />
-    </gazebo>
-    <gazebo>
-        <plugin
-            filename="gz-sim-diff-drive-system"
-            name="gz::sim::systems::DiffDrive">
-            <left_joint>left_wheel_joint</left_joint>
-            <right_joint>right_wheel_joint</right_joint>
-            <wheel_separation>0.35</wheel_separation>
-            <wheel_radius>0.1</wheel_radius>
-            <odom_publish_frequency>1</odom_publish_frequency>
-            <topic>cmd_vel</topic>
-            <odom_topic>odom</odom_topic>
-            <tf_topic>tf</tf_topic>
-            <frame_id>odom</frame_id>
-            <child_frame_id>base_link</child_frame_id>
-        </plugin>
-    </gazebo>
-    <gazebo>
-        <plugin
-            filename="gz-sim-joint-state-publisher-system"
-            name="gz::sim::systems::JointStatePublisher">
-            <topic>joint_states</topic>
-            <joint_name>left_wheel_joint</joint_name>
-            <joint_name>right_wheel_joint</joint_name>
-        </plugin>
-    </gazebo>
-</robot>
+/ros2_ws_multirobots/src/practica1/urdf/gazebo_control.xacro

File: install/practica1/share/practica1/urdf/inertial_macros.xacro (robot description, xacro)
@@ -1,32 +1 @@
-<?xml version="1.0"?>
-<robot xmlns:xacro="http://www.ros.org/wiki/xacro" >
-    <!-- Specify some standard inertial calculations https://en.wikipedia.org/wiki/List_of_moments_of_inertia -->
-    <!-- These make use of xacro's mathematical functionality -->
-    <xacro:macro name="inertial_sphere" params="mass radius *origin">
-        <inertial>
-            <xacro:insert_block name="origin"/>
-            <mass value="${mass}" />
-            <inertia ixx="${(2/5) * mass * (radius*radius)}" ixy="0.0" ixz="0.0"
-                    iyy="${(2/5) * mass * (radius*radius)}" iyz="0.0"
-                    izz="${(2/5) * mass * (radius*radius)}" />
-        </inertial>
-    </xacro:macro>
-    <xacro:macro name="inertial_box" params="mass x y z *origin">
-        <inertial>
-            <xacro:insert_block name="origin"/>
-            <mass value="${mass}" />
-            <inertia ixx="${(1/12) * mass * (y*y + z*z)}" ixy="0.0" ixz="0.0"
-                    iyy="${(1/12) * mass * (x*x + z*z)}" iyz="0.0"
-                    izz="${(1/12) * mass * (x*x + y*y)}" />
-        </inertial>
-    </xacro:macro>
-    <xacro:macro name="inertial_cylinder" params="mass length radius *origin">
-        <inertial>
-            <xacro:insert_block name="origin"/>
-            <mass value="${mass}" />
-            <inertia ixx="${(1/12) * mass * (3*radius*radius + length*length)}" ixy="0.0" ixz="0.0"
-                    iyy="${(1/12) * mass * (3*radius*radius + length*length)}" iyz="0.0"
-                    izz="${(1/2) * mass * (radius*radius)}" />
-        </inertial>
-    </xacro:macro>
-</robot>
+/ros2_ws_multirobots/src/practica1/urdf/inertial_macros.xacro

File: install/practica1/share/practica1/urdf/lidar.xacro (robot description, xacro)
@@ -1,56 +1 @@
-<?xml version="1.0"?>
-<robot xmlns:xacro="http://www.ros.org/wiki/xacro" >
-    <xacro:property name="lidar_radius" value="0.05" />
-    <xacro:property name="lidar_length" value="0.04" />
-    <xacro:property name="lidar_pkg" value="practica1" />
-    <joint name="laser_joint" type="fixed">
-        <parent link="base_link"/>
-        <child link="laser_frame"/>
-        <origin xyz="0.1 0 0.07" rpy="0 0 0"/>
-    </joint>
-    <link name="laser_frame">
-        <visual>
-            <geometry>
-                <cylinder radius="${lidar_radius}" length="${lidar_length}"/>
-            </geometry>
-            <material name="black"/>
-        </visual>
-        <collision>
-            <geometry>
-                <cylinder radius="${lidar_radius}" length="${lidar_length}"/>
-            </geometry>
-        </collision>
-        <xacro:inertial_cylinder mass="0.1" length="${lidar_length}" radius="${lidar_radius}">
-            <origin xyz="0 0 0" rpy="0 0 0"/>
-        </xacro:inertial_cylinder>
-    </link>
-    <gazebo reference="laser_frame">
-        <material>Gazebo/Black</material>
-        <sensor name="lidar" type="gpu_lidar">
-            <pose> 0 0 0 0 0 0 </pose>
-            <visualize>true</visualize>
-            <update_rate>10</update_rate>
-            <lidar>
-                <scan>
-                    <horizontal>
-                        <samples>360</samples>
-                        <resolution>1</resolution>
-                        <min_angle>-3.14</min_angle>
-                        <max_angle>3.14</max_angle>
-                    </horizontal>
-                </scan>
-                <range>
-                    <min>0.3</min>
-                    <max>12</max>
-                </range>
-                <noise>
-                  <type>gaussian</type>
-                  <mean>0.0</mean>
-                  <stddev>0.01</stddev>
-                </noise>
-            </lidar>
-            <topic>scan</topic>
-            <gz_frame_id>laser_frame</gz_frame_id>
-        </sensor>
-    </gazebo>
-</robot>
+/ros2_ws_multirobots/src/practica1/urdf/lidar.xacro

File: install/practica1/share/practica1/urdf/robotito.urdf.xacro (robot description, xacro)
@@ -1,110 +1 @@
-<?xml version="1.0"?>
-<robot name="robotito" xmlns:xacro="http://www.ros.org/wiki/xacro">
-  <!-- Include inertial macros -->
-  <xacro:include filename="inertial_macros.xacro" />
-  <xacro:include filename="gazebo_control.xacro" />
-  <xacro:include filename="lidar.xacro" />
-  <xacro:include filename="camera.xacro" />
-  <!-- Robot Properties -->
-  <xacro:property name="chassis_length" value="0.4" />
-  <xacro:property name="chassis_width" value="0.3" />
-  <xacro:property name="chassis_height" value="0.1" />
-  <xacro:property name="chassis_mass" value="1.0" />
-  <xacro:property name="wheel_radius" value="0.1" />
-  <xacro:property name="wheel_thickness" value="0.04" />
-  <xacro:property name="wheel_mass" value="0.1" />
-  <xacro:property name="wheel_offset_x" value="0.1" />
-  <xacro:property name="wheel_offset_y" value="0.1705" />
-  <xacro:property name="wheel_offset_z" value="0.0" />
-  <xacro:property name="caster_wheel_radius" value="0.025" />
-  <xacro:property name="caster_wheel_mass" value="0.05" />
-  <xacro:property name="caster_wheel_offset_x" value="0.15" />
-  <xacro:property name="caster_wheel_offset_z" value="-0.075" />
-  <!-- Materials -->
-  <material name="white">
-    <color rgba="1 1 1 1" />
-  </material>
-  <material name="orange">
-    <color rgba="1 0.3 0.1 1"/>
-  </material>
-  <material name="blue">
-    <color rgba="0.2 0.2 1 1"/>
-  </material>
-  <material name="black">
-    <color rgba="0 0 0 1"/>
-  </material>
-  <material name="green">
-    <color rgba="0 1 0 1"/>
-  </material>
-  <!-- BASE LINK -->
-  <link name="base_link">
-    <visual>
-        <origin xyz="0 0 0" rpy="0 0 0"/>
-        <geometry>
-            <box size="${chassis_length} ${chassis_width} ${chassis_height}"/>
-        </geometry>
-        <material name="green"/>
-    </visual>
-    <collision>
-        <origin xyz="0 0 0" rpy="0 0 0"/>
-        <geometry>
-            <box size="${chassis_length} ${chassis_width} ${chassis_height}"/>
-        </geometry>
-    </collision>
-    <xacro:inertial_box mass="0.5" x="${chassis_length}" y="${chassis_width}" z="${chassis_height}">
-        <origin xyz="0 0 0" rpy="0 0 0"/>
-    </xacro:inertial_box>
-  </link>
-  <!-- WHEELS -->
-  <!-- Wheel Macro -->
-  <xacro:macro name="wheel" params="prefix offset_y">
-    <link name="${prefix}_wheel">
-      <visual>
-        <origin xyz="0 0 0" rpy="1.5707 0 0 "/>
-        <geometry>
-            <cylinder radius="${wheel_radius}" length="${wheel_thickness}"/>
-        </geometry>
-        <material name="black"/>
-      </visual>
-      <collision>
-        <origin xyz="0 0 0" rpy="1.5707 0 0 "/>
-        <geometry>
-            <cylinder radius="${wheel_radius}" length="${wheel_thickness}"/>
-        </geometry>
-      </collision>
-      <xacro:inertial_cylinder mass="${wheel_mass}" length="${wheel_thickness}" radius="${wheel_radius}">
-        <origin xyz="0 0 0" rpy="1.5707 0 0"/>
-      </xacro:inertial_cylinder>
-    </link>
-    <joint name="${prefix}_wheel_joint" type="continuous">
-      <parent link="base_link"/>
-      <child link="${prefix}_wheel"/>
-      <origin xyz="${-wheel_offset_x} ${offset_y} ${wheel_offset_z}" rpy="0 0 0"/>
-      <axis xyz="0 1 0"/>
-    </joint>
-  </xacro:macro>
-  <xacro:wheel prefix="left" offset_y="${wheel_offset_y}"/>
-  <xacro:wheel prefix="right" offset_y="${-wheel_offset_y}"/>
-  <!-- CASTER WHEEL -->
-  <link name="caster_wheel">
-    <visual>
-      <geometry>
-        <sphere radius="${caster_wheel_radius}"/>
-      </geometry>
-      <material name="white"/>
-    </visual>
-    <collision>
-      <geometry>
-        <sphere radius="${caster_wheel_radius}"/>
-      </geometry>
-    </collision>
-    <xacro:inertial_sphere mass="${caster_wheel_mass}" radius="${caster_wheel_radius}">
-        <origin xyz="0 0 0" rpy="0 0 0"/>
-    </xacro:inertial_sphere>
-  </link>
-  <joint name="caster_joint" type="fixed">
-    <parent link="base_link"/>
-    <child link="caster_wheel"/>
-    <origin xyz="${caster_wheel_offset_x} 0 ${caster_wheel_offset_z}"/>
-  </joint>
-</robot>
+/ros2_ws_multirobots/src/practica1/urdf/robotito.urdf.xacro

File: src/practica1/urdf/camera.xacro (robot description, xacro)
@@ -67,6 +67,6 @@
                 </clip>
             </camera>
-            <topic>camera/image_raw</topic>
-            <gz_frame_id>camera_link_optical</gz_frame_id>
+            <topic>$(arg prefix)camera/image_raw</topic>
+            <gz_frame_id>$(arg prefix)camera_link_optical</gz_frame_id>
         </sensor>
     </gazebo>

File: src/practica1/urdf/gazebo_control.xacro (robot description, xacro)
@@ -14,9 +14,9 @@
             <wheel_radius>0.1</wheel_radius>
             <odom_publish_frequency>1</odom_publish_frequency>
-            <topic>cmd_vel</topic>
-            <odom_topic>odom</odom_topic>
-            <tf_topic>tf</tf_topic>
-            <frame_id>odom</frame_id>
-            <child_frame_id>base_link</child_frame_id>
+            <topic>$(arg prefix)cmd_vel</topic>
+            <odom_topic>$(arg prefix)odom</odom_topic>
+            <tf_topic>$(arg prefix)tf</tf_topic>
+            <frame_id>$(arg prefix)odom</frame_id>
+            <child_frame_id>$(arg prefix)base_link</child_frame_id>
         </plugin>
     </gazebo>
@@ -25,5 +25,5 @@
             filename="gz-sim-joint-state-publisher-system"
             name="gz::sim::systems::JointStatePublisher">
-            <topic>joint_states</topic>
+            <topic>$(arg prefix)joint_states</topic>
             <joint_name>left_wheel_joint</joint_name>
             <joint_name>right_wheel_joint</joint_name>

File: src/practica1/urdf/lidar.xacro (robot description, xacro)
@@ -50,6 +50,6 @@
                 </noise>
             </lidar>
-            <topic>scan</topic>
-            <gz_frame_id>laser_frame</gz_frame_id>
+            <topic>$(arg prefix)scan</topic>
+            <gz_frame_id>$(arg prefix)laser_frame</gz_frame_id>
         </sensor>
     </gazebo>

File: src/practica1/urdf/robotito.urdf.xacro (robot description, xacro)
@@ -1,4 +1,7 @@
 <?xml version="1.0"?>
 <robot name="robotito" xmlns:xacro="http://www.ros.org/wiki/xacro">
+  <!-- Namespace prefix argument (e.g. "robot1/") – empty string for single robot -->
+  <xacro:arg name="prefix" default="" />
+  <xacro:property name="ns_prefix" value="$(arg prefix)" />
   <!-- Include inertial macros -->
   <xacro:include filename="inertial_macros.xacro" />
