Commit message: lidar mas alto

File: src/practica1/urdf/lidar.xacro (robot description, xacro)
@@ -7,5 +7,5 @@
         <parent link="${ns_prefix}base_link"/>
         <child link="${ns_prefix}laser_frame"/>
-        <origin xyz="0.1 0 0.07" rpy="0 0 0"/>
+        <origin xyz="0.1 0 0.35" rpy="0 0 0"/>
     </joint>
     <link name="${ns_prefix}laser_frame">

Commit message: pos lidar corregido

File: src/practica1/urdf/lidar.xacro (robot description, xacro)
@@ -7,5 +7,5 @@
         <parent link="${ns_prefix}base_link"/>
         <child link="${ns_prefix}laser_frame"/>
-        <origin xyz="0.1 0 0.35" rpy="0 0 0"/>
+        <origin xyz="0.1 0 0.4" rpy="0 0 0"/>
     </joint>
     <link name="${ns_prefix}laser_frame">
