Commit message: base_link added for rviz2

File: src/practica1/urdf/camera.xacro (robot description, xacro)
@@ -1,10 +1,10 @@
 <?xml version="1.0"?>
 <robot xmlns:xacro="http://www.ros.org/wiki/xacro" >
-    <joint name="camera_mast_joint" type="fixed">
-        <parent link="base_link"/>
-        <child link="camera_mast"/>
+    <joint name="${ns_prefix}camera_mast_joint" type="fixed">
+        <parent link="${ns_prefix}base_link"/>
+        <child link="${ns_prefix}camera_mast"/>
         <origin xyz="0.10 0 0.20" rpy="0 0 0"/>
     </joint>
-    <link name="camera_mast">
+    <link name="${ns_prefix}camera_mast">
         <visual>
             <geometry>
@@ -22,10 +22,10 @@
         </xacro:inertial_cylinder>
     </link>
-    <joint name="camera_joint" type="fixed">
-        <parent link="camera_mast"/>
-        <child link="camera_link"/>
+    <joint name="${ns_prefix}camera_joint" type="fixed">
+        <parent link="${ns_prefix}camera_mast"/>
+        <child link="${ns_prefix}camera_link"/>
         <origin xyz="0.02 0 0.15" rpy="0 0 0"/>
     </joint>
-    <link name="camera_link">
+    <link name="${ns_prefix}camera_link">
         <visual>
             <geometry>
@@ -43,11 +43,11 @@
         </xacro:inertial_box>
     </link>
-    <joint name="camera_optical_joint" type="fixed">
+    <joint name="${ns_prefix}camera_optical_joint" type="fixed">
         <origin xyz="0 0 0" rpy="-1.5708 0 -1.5708"/>
-        <parent link="camera_link"/>
-        <child link="camera_link_optical"/>
+        <parent link="${ns_prefix}camera_link"/>
+        <child link="${ns_prefix}camera_link_optical"/>
     </joint>
-    <link name="camera_link_optical"></link>
-    <gazebo reference="camera_link">
+    <link name="${ns_prefix}camera_link_optical"></link>
+    <gazebo reference="${ns_prefix}camera_link">
         <material>Gazebo/Blue</material>
         <sensor name="camera" type="camera">

File: src/practica1/urdf/gazebo_control.xacro (robot description, xacro)
@@ -1,5 +1,5 @@
 <?xml version="1.0"?>
 <robot xmlns:xacro="http://www.ros.org/wiki/xacro">
-    <gazebo reference="caster_wheel">
+    <gazebo reference="$(arg prefix)caster_wheel">
         <mu1 value="0.1" />
         <mu2 value="0.1" />
@@ -9,6 +9,6 @@
             filename="gz-sim-diff-drive-system"
             name="gz::sim::systems::DiffDrive">
-            <left_joint>left_wheel_joint</left_joint>
-            <right_joint>right_wheel_joint</right_joint>
+            <left_joint>$(arg prefix)left_wheel_joint</left_joint>
+            <right_joint>$(arg prefix)right_wheel_joint</right_joint>
             <wheel_separation>0.35</wheel_separation>
             <wheel_radius>0.1</wheel_radius>
@@ -26,6 +26,6 @@
             name="gz::sim::systems::JointStatePublisher">
             <topic>$(arg prefix)joint_states</topic>
-            <joint_name>left_wheel_joint</joint_name>
-            <joint_name>right_wheel_joint</joint_name>
+            <joint_name>$(arg prefix)left_wheel_joint</joint_name>
+            <joint_name>$(arg prefix)right_wheel_joint</joint_name>
         </plugin>
     </gazebo>

File: src/practica1/urdf/lidar.xacro (robot description, xacro)
@@ -4,10 +4,10 @@
     <xacro:property name="lidar_length" value="0.04" />
     <xacro:property name="lidar_pkg" value="practica1" />
-    <joint name="laser_joint" type="fixed">
-        <parent link="base_link"/>
-        <child link="laser_frame"/>
+    <joint name="${ns_prefix}laser_joint" type="fixed">
+        <parent link="${ns_prefix}base_link"/>
+        <child link="${ns_prefix}laser_frame"/>
         <origin xyz="0.1 0 0.07" rpy="0 0 0"/>
     </joint>
-    <link name="laser_frame">
+    <link name="${ns_prefix}laser_frame">
         <visual>
             <geometry>
@@ -25,5 +25,5 @@
         </xacro:inertial_cylinder>
     </link>
-    <gazebo reference="laser_frame">
+    <gazebo reference="${ns_prefix}laser_frame">
         <material>Gazebo/Black</material>
         <sensor name="lidar" type="gpu_lidar">

File: src/practica1/urdf/robotito.urdf.xacro (robot description, xacro)
@@ -41,5 +41,5 @@
   </material>
   <!-- BASE LINK -->
-  <link name="base_link">
+  <link name="${ns_prefix}base_link">
     <visual>
         <origin xyz="0 0 0" rpy="0 0 0"/>
@@ -62,5 +62,5 @@
   <!-- Wheel Macro -->
   <xacro:macro name="wheel" params="prefix offset_y">
-    <link name="${prefix}_wheel">
+    <link name="${ns_prefix}${prefix}_wheel">
       <visual>
         <origin xyz="0 0 0" rpy="1.5707 0 0 "/>
@@ -80,7 +80,7 @@
       </xacro:inertial_cylinder>
     </link>
-    <joint name="${prefix}_wheel_joint" type="continuous">
-      <parent link="base_link"/>
-      <child link="${prefix}_wheel"/>
+    <joint name="${ns_prefix}${prefix}_wheel_joint" type="continuous">
+      <parent link="${ns_prefix}base_link"/>
+      <child link="${ns_prefix}${prefix}_wheel"/>
       <origin xyz="${-wheel_offset_x} ${offset_y} ${wheel_offset_z}" rpy="0 0 0"/>
       <axis xyz="0 1 0"/>
@@ -90,5 +90,5 @@
   <xacro:wheel prefix="right" offset_y="${-wheel_offset_y}"/>
   <!-- CASTER WHEEL -->
-  <link name="caster_wheel">
+  <link name="${ns_prefix}caster_wheel">
     <visual>
       <geometry>
@@ -106,7 +106,7 @@
     </xacro:inertial_sphere>
   </link>
-  <joint name="caster_joint" type="fixed">
-    <parent link="base_link"/>
-    <child link="caster_wheel"/>
+  <joint name="${ns_prefix}caster_joint" type="fixed">
+    <parent link="${ns_prefix}base_link"/>
+    <child link="${ns_prefix}caster_wheel"/>
     <origin xyz="${caster_wheel_offset_x} 0 ${caster_wheel_offset_z}"/>
   </joint>

Commit message: mejorada legibilidad de variables

File: src/practica1/urdf/camera.xacro (robot description, xacro)
@@ -1,10 +1,10 @@
 <?xml version="1.0"?>
 <robot xmlns:xacro="http://www.ros.org/wiki/xacro" >
-    <joint name="${ns_prefix}camera_mast_joint" type="fixed">
-        <parent link="${ns_prefix}base_link"/>
-        <child link="${ns_prefix}camera_mast"/>
+    <joint name="${prefijo_ns}camera_mast_joint" type="fixed">
+        <parent link="${prefijo_ns}base_link"/>
+        <child link="${prefijo_ns}camera_mast"/>
         <origin xyz="0.10 0 0.20" rpy="0 0 0"/>
     </joint>
-    <link name="${ns_prefix}camera_mast">
+    <link name="${prefijo_ns}camera_mast">
         <visual>
             <geometry>
@@ -22,10 +22,10 @@
         </xacro:inertial_cylinder>
     </link>
-    <joint name="${ns_prefix}camera_joint" type="fixed">
-        <parent link="${ns_prefix}camera_mast"/>
-        <child link="${ns_prefix}camera_link"/>
+    <joint name="${prefijo_ns}camera_joint" type="fixed">
+        <parent link="${prefijo_ns}camera_mast"/>
+        <child link="${prefijo_ns}camera_link"/>
         <origin xyz="0.02 0 0.15" rpy="0 0 0"/>
     </joint>
-    <link name="${ns_prefix}camera_link">
+    <link name="${prefijo_ns}camera_link">
         <visual>
             <geometry>
@@ -43,11 +43,11 @@
         </xacro:inertial_box>
     </link>
-    <joint name="${ns_prefix}camera_optical_joint" type="fixed">
+    <joint name="${prefijo_ns}camera_optical_joint" type="fixed">
         <origin xyz="0 0 0" rpy="-1.5708 0 -1.5708"/>
-        <parent link="${ns_prefix}camera_link"/>
-        <child link="${ns_prefix}camera_link_optical"/>
+        <parent link="${prefijo_ns}camera_link"/>
+        <child link="${prefijo_ns}camera_link_optical"/>
     </joint>
-    <link name="${ns_prefix}camera_link_optical"></link>
-    <gazebo reference="${ns_prefix}camera_link">
+    <link name="${prefijo_ns}camera_link_optical"></link>
+    <gazebo reference="${prefijo_ns}camera_link">
         <material>Gazebo/Blue</material>
         <sensor name="camera" type="camera">

File: src/practica1/urdf/inertial_macros.xacro (robot description, xacro)
@@ -1,6 +1,4 @@
 <?xml version="1.0"?>
 <robot xmlns:xacro="http://www.ros.org/wiki/xacro" >
-    <!-- Specify some standard inertial calculations https://en.wikipedia.org/wiki/List_of_moments_of_inertia -->
-    <!-- These make use of xacro's mathematical functionality -->
     <xacro:macro name="inertial_sphere" params="mass radius *origin">
         <inertial>

File: src/practica1/urdf/lidar.xacro (robot description, xacro)
@@ -1,16 +1,16 @@
 <?xml version="1.0"?>
 <robot xmlns:xacro="http://www.ros.org/wiki/xacro" >
-    <xacro:property name="lidar_radius" value="0.05" />
-    <xacro:property name="lidar_length" value="0.04" />
-    <xacro:property name="lidar_pkg" value="practica1" />
-    <joint name="${ns_prefix}laser_joint" type="fixed">
-        <parent link="${ns_prefix}base_link"/>
-        <child link="${ns_prefix}laser_frame"/>
+    <xacro:property name="radio_lidar" value="0.05" />
+    <xacro:property name="longitud_lidar" value="0.04" />
+    <xacro:property name="paquete_lidar" value="practica1" />
+    <joint name="${prefijo_ns}laser_joint" type="fixed">
+        <parent link="${prefijo_ns}base_link"/>
+        <child link="${prefijo_ns}laser_frame"/>
         <origin xyz="0.1 0 0.4" rpy="0 0 0"/>
     </joint>
-    <link name="${ns_prefix}laser_frame">
+    <link name="${prefijo_ns}laser_frame">
         <visual>
             <geometry>
-                <cylinder radius="${lidar_radius}" length="${lidar_length}"/>
+                <cylinder radius="${radio_lidar}" length="${longitud_lidar}"/>
             </geometry>
             <material name="black"/>
@@ -18,12 +18,12 @@
         <collision>
             <geometry>
-                <cylinder radius="${lidar_radius}" length="${lidar_length}"/>
+                <cylinder radius="${radio_lidar}" length="${longitud_lidar}"/>
             </geometry>
         </collision>
-        <xacro:inertial_cylinder mass="0.1" length="${lidar_length}" radius="${lidar_radius}">
+        <xacro:inertial_cylinder mass="0.1" length="${longitud_lidar}" radius="${radio_lidar}">
             <origin xyz="0 0 0" rpy="0 0 0"/>
         </xacro:inertial_cylinder>
     </link>
-    <gazebo reference="${ns_prefix}laser_frame">
+    <gazebo reference="${prefijo_ns}laser_frame">
         <material>Gazebo/Black</material>
         <sensor name="lidar" type="gpu_lidar">
@@ -41,6 +41,6 @@
                 </scan>
                 <range>
-                    <min>0.3</min>
-                    <max>12</max>
+                    <min>0.1</min>
+                    <max>10</max> <!-- 12 metros por ejemplo de max -->
                 </range>
                 <noise>

File: src/practica1/urdf/robotito.urdf.xacro (robot description, xacro)
@@ -1,28 +1,27 @@
 <?xml version="1.0"?>
 <robot name="robotito" xmlns:xacro="http://www.ros.org/wiki/xacro">
-  <!-- Namespace prefix argument (e.g. "robot1/") – empty string for single robot -->
+  <!-- namespace -->
   <xacro:arg name="prefix" default="" />
-  <xacro:property name="ns_prefix" value="$(arg prefix)" />
-  <!-- Include inertial macros -->
+  <xacro:property name="prefijo_ns" value="$(arg prefix)" />
+  <!-- los distintos archivos que usa -->
   <xacro:include filename="inertial_macros.xacro" />
   <xacro:include filename="gazebo_control.xacro" />
   <xacro:include filename="lidar.xacro" />
   <xacro:include filename="camera.xacro" />
-  <!-- Robot Properties -->
-  <xacro:property name="chassis_length" value="0.4" />
-  <xacro:property name="chassis_width" value="0.3" />
-  <xacro:property name="chassis_height" value="0.1" />
-  <xacro:property name="chassis_mass" value="1.0" />
-  <xacro:property name="wheel_radius" value="0.1" />
-  <xacro:property name="wheel_thickness" value="0.04" />
-  <xacro:property name="wheel_mass" value="0.1" />
-  <xacro:property name="wheel_offset_x" value="0.1" />
-  <xacro:property name="wheel_offset_y" value="0.1705" />
-  <xacro:property name="wheel_offset_z" value="0.0" />
-  <xacro:property name="caster_wheel_radius" value="0.025" />
-  <xacro:property name="caster_wheel_mass" value="0.05" />
-  <xacro:property name="caster_wheel_offset_x" value="0.15" />
-  <xacro:property name="caster_wheel_offset_z" value="-0.075" />
-  <!-- Materials -->
+  <!-- ya las cosas del robot -->
+  <xacro:property name="largo_chasis" value="0.4" />
+  <xacro:property name="ancho_chasis" value="0.3" />
+  <xacro:property name="alto_chasis" value="0.1" />
+  <xacro:property name="masa_chasis" value="1.0" />
+  <xacro:property name="radio_rueda" value="0.1" />
+  <xacro:property name="grosor_rueda" value="0.04" />
+  <xacro:property name="masa_rueda" value="0.1" />
+  <xacro:property name="offset_rueda_x" value="0.1" />
+  <xacro:property name="offset_rueda_y" value="0.1705" />
+  <xacro:property name="offset_rueda_z" value="0.0" />
+  <xacro:property name="radio_rueda_loca" value="0.025" />
+  <xacro:property name="masa_rueda_loca" value="0.05" />
+  <xacro:property name="offset_rueda_loca_x" value="0.15" />
+  <xacro:property name="offset_rueda_loca_z" value="-0.075" />
   <material name="white">
     <color rgba="1 1 1 1" />
@@ -40,10 +39,10 @@
     <color rgba="0 1 0 1"/>
   </material>
-  <!-- BASE LINK -->
-  <link name="${ns_prefix}base_link">
+  <!-- el base link-->
+  <link name="${prefijo_ns}base_link">
     <visual>
         <origin xyz="0 0 0" rpy="0 0 0"/>
         <geometry>
-            <box size="${chassis_length} ${chassis_width} ${chassis_height}"/>
+            <box size="${largo_chasis} ${ancho_chasis} ${alto_chasis}"/>
         </geometry>
         <material name="green"/>
@@ -52,19 +51,18 @@
         <origin xyz="0 0 0" rpy="0 0 0"/>
         <geometry>
-            <box size="${chassis_length} ${chassis_width} ${chassis_height}"/>
+            <box size="${largo_chasis} ${ancho_chasis} ${alto_chasis}"/>
         </geometry>
     </collision>
-    <xacro:inertial_box mass="0.5" x="${chassis_length}" y="${chassis_width}" z="${chassis_height}">
+    <xacro:inertial_box mass="${masa_chasis}" x="${largo_chasis}" y="${ancho_chasis}" z="${alto_chasis}">
         <origin xyz="0 0 0" rpy="0 0 0"/>
     </xacro:inertial_box>
   </link>
-  <!-- WHEELS -->
-  <!-- Wheel Macro -->
-  <xacro:macro name="wheel" params="prefix offset_y">
-    <link name="${ns_prefix}${prefix}_wheel">
+  <!-- wheel macro -->
+  <xacro:macro name="wheel" params="lado desplazamiento_y">
+    <link name="${prefijo_ns}${lado}_wheel">
       <visual>
         <origin xyz="0 0 0" rpy="1.5707 0 0 "/>
         <geometry>
-            <cylinder radius="${wheel_radius}" length="${wheel_thickness}"/>
+            <cylinder radius="${radio_rueda}" length="${grosor_rueda}"/>
         </geometry>
         <material name="black"/>
@@ -73,25 +71,25 @@
         <origin xyz="0 0 0" rpy="1.5707 0 0 "/>
         <geometry>
-            <cylinder radius="${wheel_radius}" length="${wheel_thickness}"/>
+            <cylinder radius="${radio_rueda}" length="${grosor_rueda}"/>
         </geometry>
       </collision>
-      <xacro:inertial_cylinder mass="${wheel_mass}" length="${wheel_thickness}" radius="${wheel_radius}">
+      <xacro:inertial_cylinder mass="${masa_rueda}" length="${grosor_rueda}" radius="${radio_rueda}">
         <origin xyz="0 0 0" rpy="1.5707 0 0"/>
       </xacro:inertial_cylinder>
     </link>
-    <joint name="${ns_prefix}${prefix}_wheel_joint" type="continuous">
-      <parent link="${ns_prefix}base_link"/>
-      <child link="${ns_prefix}${prefix}_wheel"/>
-      <origin xyz="${-wheel_offset_x} ${offset_y} ${wheel_offset_z}" rpy="0 0 0"/>
+    <joint name="${prefijo_ns}${lado}_wheel_joint" type="continuous">
+      <parent link="${prefijo_ns}base_link"/>
+      <child link="${prefijo_ns}${lado}_wheel"/>
+      <origin xyz="${-offset_rueda_x} ${desplazamiento_y} ${offset_rueda_z}" rpy="0 0 0"/>
       <axis xyz="0 1 0"/>
     </joint>
   </xacro:macro>
-  <xacro:wheel prefix="left" offset_y="${wheel_offset_y}"/>
-  <xacro:wheel prefix="right" offset_y="${-wheel_offset_y}"/>
-  <!-- CASTER WHEEL -->
-  <link name="${ns_prefix}caster_wheel">
+  <xacro:wheel lado="left" desplazamiento_y="${offset_rueda_y}"/>
+  <xacro:wheel lado="right" desplazamiento_y="${-offset_rueda_y}"/>
+<!-- rueda caster-->
+  <link name="${prefijo_ns}caster_wheel">
     <visual>
       <geometry>
-        <sphere radius="${caster_wheel_radius}"/>
+        <sphere radius="${radio_rueda_loca}"/>
       </geometry>
       <material name="white"/>
@@ -99,15 +97,15 @@
     <collision>
       <geometry>
-        <sphere radius="${caster_wheel_radius}"/>
+        <sphere radius="${radio_rueda_loca}"/>
       </geometry>
     </collision>
-    <xacro:inertial_sphere mass="${caster_wheel_mass}" radius="${caster_wheel_radius}">
+    <xacro:inertial_sphere mass="${masa_rueda_loca}" radius="${radio_rueda_loca}">
         <origin xyz="0 0 0" rpy="0 0 0"/>
     </xacro:inertial_sphere>
   </link>
-  <joint name="${ns_prefix}caster_joint" type="fixed">
-    <parent link="${ns_prefix}base_link"/>
-    <child link="${ns_prefix}caster_wheel"/>
-    <origin xyz="${caster_wheel_offset_x} 0 ${caster_wheel_offset_z}"/>
+  <joint name="${prefijo_ns}caster_joint" type="fixed">
+    <parent link="${prefijo_ns}base_link"/>
+    <child link="${prefijo_ns}caster_wheel"/>
+    <origin xyz="${offset_rueda_loca_x} 0 ${offset_rueda_loca_z}"/>
   </joint>
 </robot>

Commit message: mejorada legibilidad de variables

File: src/practica1/urdf/camera.xacro (robot description, xacro)
@@ -18,7 +18,7 @@
             </geometry>
         </collision>
-        <xacro:inertial_cylinder mass="0.05" length="0.30" radius="0.02">
+        <xacro:inercia_cilindro mass="0.05" length="0.30" radius="0.02">
             <origin xyz="0 0 0" rpy="0 0 0"/>
-        </xacro:inertial_cylinder>
+        </xacro:inercia_cilindro>
     </link>
     <joint name="${prefijo_ns}camera_joint" type="fixed">
@@ -39,7 +39,7 @@
             </geometry>
         </collision>
-        <xacro:inertial_box mass="0.05" x="0.05" y="0.05" z="0.05">
+        <xacro:inercia_caja mass="0.05" x="0.05" y="0.05" z="0.05">
             <origin xyz="0 0 0" rpy="0 0 0"/>
-        </xacro:inertial_box>
+        </xacro:inercia_caja>
     </link>
     <joint name="${prefijo_ns}camera_optical_joint" type="fixed">

File: src/practica1/urdf/inertial_macros.xacro (robot description, xacro)
@@ -1,5 +1,5 @@
 <?xml version="1.0"?>
 <robot xmlns:xacro="http://www.ros.org/wiki/xacro" >
-    <xacro:macro name="inertial_sphere" params="mass radius *origin">
+    <xacro:macro name="inercia_esfera" params="mass radius *origin">
         <inertial>
             <xacro:insert_block name="origin"/>
@@ -10,5 +10,5 @@
         </inertial>
     </xacro:macro>
-    <xacro:macro name="inertial_box" params="mass x y z *origin">
+    <xacro:macro name="inercia_caja" params="mass x y z *origin">
         <inertial>
             <xacro:insert_block name="origin"/>
@@ -19,5 +19,5 @@
         </inertial>
     </xacro:macro>
-    <xacro:macro name="inertial_cylinder" params="mass length radius *origin">
+    <xacro:macro name="inercia_cilindro" params="mass length radius *origin">
         <inertial>
             <xacro:insert_block name="origin"/>

File: src/practica1/urdf/lidar.xacro (robot description, xacro)
@@ -21,7 +21,7 @@
             </geometry>
         </collision>
-        <xacro:inertial_cylinder mass="0.1" length="${longitud_lidar}" radius="${radio_lidar}">
+        <xacro:inercia_cilindro mass="0.1" length="${longitud_lidar}" radius="${radio_lidar}">
             <origin xyz="0 0 0" rpy="0 0 0"/>
-        </xacro:inertial_cylinder>
+        </xacro:inercia_cilindro>
     </link>
     <gazebo reference="${prefijo_ns}laser_frame">

File: src/practica1/urdf/robotito.urdf.xacro (robot description, xacro)
@@ -54,7 +54,7 @@
         </geometry>
     </collision>
-    <xacro:inertial_box mass="${masa_chasis}" x="${largo_chasis}" y="${ancho_chasis}" z="${alto_chasis}">
+    <xacro:inercia_caja mass="${masa_chasis}" x="${largo_chasis}" y="${ancho_chasis}" z="${alto_chasis}">
         <origin xyz="0 0 0" rpy="0 0 0"/>
-    </xacro:inertial_box>
+    </xacro:inercia_caja>
   </link>
   <!-- wheel macro -->
@@ -74,7 +74,7 @@
         </geometry>
       </collision>
-      <xacro:inertial_cylinder mass="${masa_rueda}" length="${grosor_rueda}" radius="${radio_rueda}">
+      <xacro:inercia_cilindro mass="${masa_rueda}" length="${grosor_rueda}" radius="${radio_rueda}">
         <origin xyz="0 0 0" rpy="1.5707 0 0"/>
-      </xacro:inertial_cylinder>
+      </xacro:inercia_cilindro>
     </link>
     <joint name="${prefijo_ns}${lado}_wheel_joint" type="continuous">
@@ -100,7 +100,7 @@
       </geometry>
     </collision>
-    <xacro:inertial_sphere mass="${masa_rueda_loca}" radius="${radio_rueda_loca}">
+    <xacro:inercia_esfera mass="${masa_rueda_loca}" radius="${radio_rueda_loca}">
         <origin xyz="0 0 0" rpy="0 0 0"/>
-    </xacro:inertial_sphere>
+    </xacro:inercia_esfera>
   </link>
   <joint name="${prefijo_ns}caster_joint" type="fixed">
